File: flight-computer/dino/batt-div.sch (KiCad schematic (older format))
At the start: 3 parts

Commit message: fc pinout and component selection. general cleanup
Parts:
- R?: footprint (none) -> Resistor_SMD:R_0603_1608Metric; LCSC (none) -> C23189
- R?: footprint (none) -> Resistor_SMD:R_0603_1608Metric; LCSC (none) -> C21190
Changed lines of the file:
@@
 $Descr A 11000 8500
 encoding utf-8
-Sheet 7 14
+Sheet 12 14
 Title ""
 Date ""
@@
 AR Path="/61C27E7D/61DC5AA2/61DB7284" Ref="R?"  Part="1"
 AR Path="/61D7382A/61DC5AA2/61DB7284" Ref="R?"  Part="1"
+AR Path="/61C15AA8/61E6D56F/61DB7284" Ref="R?"  Part="1"
+AR Path="/61C27F52/61E6D56F/61DB7284" Ref="R?"  Part="1"
+AR Path="/61D7382A/61E6D56F/61DB7284" Ref="R?"  Part="1"
+AR Path="/61C27E7D/61E6D56F/61DB7284" Ref="R?"  Part="1"
+AR Path="/61F91E79/61DC5AA2/61DB7284" Ref="R?"  Part="1"
+AR Path="/61F965DC/61DC5AA2/61DB7284" Ref="R?"  Part="1"
+AR Path="/61F965E7/61DC5AA2/61DB7284" Ref="R?"  Part="1"
 F 0 "R?" H 5120 3996 50  0000 L CNN
 F 1 "5k6" H 5120 3905 50  0000 L CNN
-F 2 "" V 4980 3950 50  0001 C CNN
+F 2 "Resistor_SMD:R_0603_1608Metric" V 4980 3950 50  0001 C CNN
 F 3 "~" H 5050 3950 50  0001 C CNN
+F 4 "C23189" H 5050 3950 50  0001 C CNN "LCSC"
 	1    5050 3950
 	1    0    0    -1
@@
 AR Path="/61C27E7D/61DC5AA2/61DB728A" Ref="R?"  Part="1"
 AR Path="/61D7382A/61DC5AA2/61DB728A" Ref="R?"  Part="1"
+AR Path="/61C15AA8/61E6D56F/61DB728A" Ref="R?"  Part="1"
+AR Path="/61C27F52/61E6D56F/61DB728A" Ref="R?"  Part="1"
+AR Path="/61D7382A/61E6D56F/61DB728A" Ref="R?"  Part="1"
+AR Path="/61C27E7D/61E6D56F/61DB728A" Ref="R?"  Part="1"
+AR Path="/61F91E79/61DC5AA2/61DB728A" Ref="R?"  Part="1"
+AR Path="/61F965DC/61DC5AA2/61DB728A" Ref="R?"  Part="1"
+AR Path="/61F965E7/61DC5AA2/61DB728A" Ref="R?"  Part="1"
 F 0 "R?" H 5120 4396 50  0000 L CNN
 F 1 "1k" H 5120 4305 50  0000 L CNN
-F 2 "" V 4980 4350 50  0001 C CNN
+F 2 "Resistor_SMD:R_0603_1608Metric" V 4980 4350 50  0001 C CNN
 F 3 "~" H 5050 4350 50  0001 C CNN
+F 4 "C21190" H 5050 4350 50  0001 C CNN "LCSC"
 	1    5050 4350
 	1    0    0    -1
@@
 AR Path="/61C27E7D/61DC5AA2/61DB7291" Ref="#PWR?"  Part="1"
 AR Path="/61D7382A/61DC5AA2/61DB7291" Ref="#PWR?"  Part="1"
+AR Path="/61C15AA8/61E6D56F/61DB7291" Ref="#PWR?"  Part="1"
+AR Path="/61C27F52/61E6D56F/61DB7291" Ref="#PWR?"  Part="1"
+AR Path="/61D7382A/61E6D56F/61DB7291" Ref="#PWR?"  Part="1"
+AR Path="/61C27E7D/61E6D56F/61DB7291" Ref="#PWR?"  Part="1"
+AR Path="/61F91E79/61DC5AA2/61DB7291" Ref="#PWR?"  Part="1"
+AR Path="/61F965DC/61DC5AA2/61DB7291" Ref="#PWR?"  Part="1"
+AR Path="/61F965E7/61DC5AA2/61DB7291" Ref="#PWR?"  Part="1"
 F 0 "#PWR?" H 5050 4350 50  0001 C CNN
 F 1 "GND" H 5055 4427 50  0000 C CNN
@@
 AR Path="/61C27E7D/61DC5AA2/61DB72A2" Ref="D?"  Part="1"
 AR Path="/61D7382A/61DC5AA2/61DB72A2" Ref="D?"  Part="1"
+AR Path="/61C15AA8/61E6D56F/61DB72A2" Ref="D?"  Part="1"
+AR Path="/61C27F52/61E6D56F/61DB72A2" Ref="D?"  Part="1"
+AR Path="/61D7382A/61E6D56F/61DB72A2" Ref="D?"  Part="1"
+AR Path="/61C27E7D/61E6D56F/61DB72A2" Ref="D?"  Part="1"
+AR Path="/61F91E79/61DC5AA2/61DB72A2" Ref="D?"  Part="1"
+AR Path="/61F965DC/61DC5AA2/61DB72A2" Ref="D?"  Part="1"
+AR Path="/61F965E7/61DC5AA2/61DB72A2" Ref="D?"  Part="1"
 F 0 "D?" V 5354 4429 50  0000 L CNN
 F 1 "Zener 3V3, 5%" V 5445 4429 50  0000 L CNN
